File: pcb/Carte_puissance/Carte_puissance.sch (KiCad schematic (older format))
At the start: 37 parts, among them J1 Conn_01x02, J2 Conn_02x07_Odd_Even, J3 Conn_02x04_Odd_Even, J4 MOT LEFT, J5 MOT RIGHT, J6 Conn_01x03, Q1 IPD50P04P4-13, SW1 SW_SPDT, U1 IFX9202ED, U2 MIC29500-3.3WT, U3 MIC29500-5.0WT

Commit message: Cartes En cours de conception
Parts:
- removed J3: Conn_02x04_Odd_Even, Connector_PinHeader_2.54mm:PinHeader_2x04_P2.54mm_Vertical, symbol Connector_Generic:Conn_02x04_Odd_Even
- added J3: Molex KK 254, Connector_Molex:Molex_KK-254_AE-6410-04A_1x04_P2.54mm_Vertical, symbol Connector_Generic:Conn_01x04
- FB1, FB2: footprint Capacitor_SMD:C_2220_5650Metric_Pad1.97x5.40mm_HandSolder -> Capacitor_SMD:C_1812_4532Metric_Pad1.30x3.40mm_HandSolder
Connections:
- wire segments 157 -> 150
Other:
- note added: "Courant a vide (8.4V): 0.48A"
- note added: "Courant de court circuit: >5A\nCourant en forte charge: Env 3A\nCourant en charge (sur voiture): Env 1.5A à 2A"
- note added: "IC candidat: TI DRV8873 (Pont en H, 10A)\n ST VNH5050A-E (Demi pont, 30A)\n Infineon IFX9202ED (Double pont H, 6A chaque)"
- note added: "Moteur type mabuchi 280"
Changed lines of the file:
@@
 L power:GND #PWR0113
 U 1 1 5D391944
-P 10200 2150
-F 0 "#PWR0113" H 10200 1900 50  0001 C CNN
-F 1 "GND" H 10205 1977 50  0000 C CNN
-F 2 "" H 10200 2150 50  0001 C CNN
-F 3 "" H 10200 2150 50  0001 C CNN
-	1    10200 2150
+P 9400 2100
+F 0 "#PWR0113" H 9400 1850 50  0001 C CNN
+F 1 "GND" H 9405 1927 50  0000 C CNN
+F 2 "" H 9400 2100 50  0001 C CNN
+F 3 "" H 9400 2100 50  0001 C CNN
+	1    9400 2100
 	1    0    0    -1
 $EndComp
@@
 	1    0    0    -1
 $EndComp
-Wire Wire Line
-	10000 1700 10200 1700
 Wire Wire Line
 	7250 1900 6700 1900
@@
 OUT_1_MOT_R
 Wire Wire Line
-	10200 1700 10200 1800
-Wire Wire Line
 	9500 1500 9500 1150
 $Comp
@@
 	1    0    0    -1
 $EndComp
-Wire Wire Line
-	10000 1500 10200 1500
-Wire Wire Line
-	10200 1500 10200 1600
-Connection ~ 10200 1700
-Wire Wire Line
-	10000 1600 10200 1600
-Connection ~ 10200 1600
-Wire Wire Line
-	10200 1600 10200 1700
-Wire Wire Line
-	9300 1150 9300 1600
-Wire Wire Line
-	9300 1700 9500 1700
-Wire Wire Line
-	9500 1600 9300 1600
-Connection ~ 9300 1600
-Wire Wire Line
-	9300 1600 9300 1700
 $Comp
 L Insa:MIC29500-3.3WT U2
@@
 	1    0    0    -1
 $EndComp
-$Comp
-L Connector_Generic:Conn_02x04_Odd_Even J3
-U 1 1 5D38A3E4
-P 9700 1600
-F 0 "J3" H 9750 1825 50  0000 C CNN
-F 1 "Conn_02x04_Odd_Even" H 9750 1826 50  0001 C CNN
-F 2 "Connector_PinHeader_2.54mm:PinHeader_2x04_P2.54mm_Vertical" H 9700 1600 50  0001 C CNN
-F 3 "~" H 9700 1600 50  0001 C CNN
-	1    9700 1600
-	1    0    0    -1
-$EndComp
-Connection ~ 10200 1800
-Wire Wire Line
-	10200 1800 10200 2150
-Wire Wire Line
-	9500 1800 9300 1800
-Wire Wire Line
-	9300 1800 9300 1700
-Connection ~ 9300 1700
-Wire Wire Line
-	10000 1800 10200 1800
 Wire Wire Line
 	6750 3300 6500 3300
@@
 F 0 "FB1" V 3668 1500 50  0000 C CNN
 F 1 "Ferrite_Bead" V 3667 1500 50  0001 C CNN
-F 2 "Capacitor_SMD:C_2220_5650Metric_Pad1.97x5.40mm_HandSolder" V 3780 1500 50  0001 C CNN
+F 2 "Capacitor_SMD:C_1812_4532Metric_Pad1.30x3.40mm_HandSolder" V 3780 1500 50  0001 C CNN
 F 3 "~" H 3850 1500 50  0001 C CNN
 	1    3850 1500
@@
 F 0 "FB2" V 8068 3300 50  0000 C CNN
 F 1 "Ferrite_Bead" V 8067 3300 50  0001 C CNN
-F 2 "Capacitor_SMD:C_2220_5650Metric_Pad1.97x5.40mm_HandSolder" V 8180 3300 50  0001 C CNN
+F 2 "Capacitor_SMD:C_1812_4532Metric_Pad1.30x3.40mm_HandSolder" V 8180 3300 50  0001 C CNN
 F 3 "~" H 8250 3300 50  0001 C CNN
 	1    8250 3300
@@
 	7850 6050 7850 6150
 Connection ~ 7850 6050
+$Comp
+L Connector_Generic:Conn_01x04 J3
+U 1 1 5D41F135
+P 9800 1600
+F 0 "J3" H 9880 1592 50  0000 L CNN
+F 1 "Molex KK 254" H 9880 1501 50  0000 L CNN
+F 2 "Connector_Molex:Molex_KK-254_AE-6410-04A_1x04_P2.54mm_Vertical" H 9800 1600 50  0001 C CNN
+F 3 "~" H 9800 1600 50  0001 C CNN
+	1    9800 1600
+	1    0    0    -1
+$EndComp
+Wire Wire Line
+	9300 1150 9300 1700
+Wire Wire Line
+	9600 1600 9400 1600
+Wire Wire Line
+	9400 1600 9400 1800
+Wire Wire Line
+	9600 1800 9400 1800
+Connection ~ 9400 1800
+Wire Wire Line
+	9400 1800 9400 2100
+Wire Wire Line
+	9300 1700 9600 1700
+Wire Wire Line
+	9500 1500 9600 1500
+Text Notes 750  2900 0    50   ~ 0
+Moteur type mabuchi 280
+Text Notes 750  3000 0    50   ~ 0
+Courant a vide (8.4V): 0.48A
+Text Notes 750  3250 0    50   ~ 0
+Courant de court circuit: >5A\nCourant en forte charge: Env 3A\nCourant en charge (sur voiture): Env 1.5A à 2A
+Text Notes 750  3550 0    50   ~ 0
+IC candidat: TI DRV8873 (Pont en H, 10A)\n              ST VNH5050A-E (Demi pont, 30A)\n              Infineon IFX9202ED (Double pont H, 6A chaque)
 $EndSCHEMATC

Commit message: demarrage carte capteurs
Parts:
- removed H1, H3: MountingHole, MountingHole:MountingHole_3.2mm_M3, symbol Mechanical:MountingHole
- removed U1: IFX9202ED, Insa:Infineon_PG_DSO_36, symbol Insa:IFX9202ED
- added C12, C15: 1nF, Capacitor_SMD:C_1206_3216Metric_Pad1.42x1.75mm_HandSolder, symbol Device:C
- added C13, C14, C16, C17, C22: 100nF, Capacitor_SMD:C_1206_3216Metric_Pad1.42x1.75mm_HandSolder, symbol Device:C
- added C23: 470µF, Capacitor_THT:CP_Radial_D6.3mm_P2.50mm, symbol Device:CP
- added Q2, Q3, Q4, Q5: BTN8982TA, Package_TO_SOT_SMD:TO-263-7_TabPin8, symbol Power_Management:BTN8982TA
- added R10, R11, R12, R5, R6, R7, R8, R9: 10K, Resistor_SMD:R_1206_3216Metric_Pad1.42x1.75mm_HandSolder, symbol Device:R
- added R13, R16: 1K, Resistor_SMD:R_1206_3216Metric_Pad1.42x1.75mm_HandSolder, symbol Device:R
- added R14, R15, R17, R18: 510R, Resistor_SMD:R_1206_3216Metric_Pad1.42x1.75mm_HandSolder, symbol Device:R
- C20: renamed from C2; value 100µF -> 470µF
- renumbered C6 to C1, C1 to C19, C3 to C2, C4 to C3, C5 to C4, C7 to C5, H2 to H1, H4 to H2
Connections:
- net labels added: FEEDBACK_MOT_L, FEEDBACK_MOT_R, PWM_MOT_L_1, PWM_MOT_L_2, PWM_MOT_R_1, PWM_MOT_R_2
- net labels removed: DIR_MOT_L, DIR_MOT_R, MISO_MOT_DRV, MOSI_MOT_DRV, PWM_MOT_L, PWM_MOT_R, SCK_MOT_DRV, ~CS_SPI_MOT_LEFT, ~CS_SPI_MOT_RIGHT
- wire segments 150 -> 189
- no-connect marks 0 -> 2
Other:
- note added: "IC candidat: TI DRV8873 (Pont en H, 10A)\n ST VNH5050A-E (Demi pont, 30A)\n Infineon IFX9202ED (Double pont H, 6A chaque)\n Infineon BTN8962TA (Half Bridge 30A)"
- note removed: "IC candidat: TI DRV8873 (Pont en H, 10A)\n ST VNH5050A-E (Demi pont, 30A)\n Infineon IFX9202ED (Double pont H, 6A chaque)"
- moved on the sheet: C19, C20, H1, H2, J3

Commit message: ajout des versions sur les cartes
Parts:
- added C6: 100nF, Capacitor_SMD:C_1206_3216Metric_Pad1.42x1.75mm_HandSolder, symbol Device:C
- renumbered H1 to H4
Connections:
- net +5V: now also C6.2
- net GNDA: now also C6.1
Changed lines of the file:
@@
 EESchema Schematic File Version 4
 LIBS:Carte_puissance-cache
-EELAYER 26 0
+EELAYER 30 0
 EELAYER END
 $Descr A4 11693 8268
@@
 	10050 4900 9800 4900
 Wire Wire Line
-	9800 4900 9800 5150
+	9800 4900 9800 5100
 Wire Wire Line
 	10050 4700 9100 4700
@@
 $EndComp
 $Comp
-L Mechanical:MountingHole H1
+L Mechanical:MountingHole H4
 U 1 1 5D5DDCC8
 P 850 7450
-F 0 "H1" H 950 7450 50  0000 L CNN
+F 0 "H4" H 950 7450 50  0000 L CNN
 F 1 "MountingHole" H 950 7405 50  0001 L CNN
 F 2 "MountingHole:MountingHole_3.2mm_M3" H 850 7450 50  0001 C CNN
@@
 	1    0    0    -1
 $EndComp
+$Comp
+L Device:C C6
+U 1 1 5D71DB77
+P 9600 4950
+F 0 "C6" H 9715 4996 50  0000 L CNN
+F 1 "100nF" H 9715 4905 50  0000 L CNN
+F 2 "Capacitor_SMD:C_1206_3216Metric_Pad1.42x1.75mm_HandSolder" H 9638 4800 50  0001 C CNN
+F 3 "~" H 9600 4950 50  0001 C CNN
+	1    9600 4950
+	-1   0    0    1
+$EndComp
+Wire Wire Line
+	9800 4800 9600 4800
+Connection ~ 9800 4800
+Wire Wire Line
+	9600 5100 9800 5100
+Connection ~ 9800 5100
+Wire Wire Line
+	9800 5100 9800 5150
 $EndSCHEMATC

Commit message: Correction sur carte capteur + realisation des pieces du circuit sous LibreCad/InkScape
Parts:
- C20, C23: value 470µF -> 100µF
- R2: value 330R -> 470R
- R3: value 330R -> 220R
- R4: value 330R -> 100R
Other:
- note added: "TODO: Rajouter des resistances de pulldown sur les entrées IN des BTN8982TA"
Changed lines of the file:
@@
 P 4400 7200
 F 0 "C20" H 4518 7246 50  0000 L CNN
-F 1 "470µF" H 4518 7155 50  0000 L CNN
+F 1 "100µF" H 4518 7155 50  0000 L CNN
 F 2 "Capacitor_THT:CP_Radial_D6.3mm_P2.50mm" H 4438 7050 50  0001 C CNN
 F 3 "~" H 4400 7200 50  0001 C CNN
@@
 P 4950 1850
 F 0 "R2" H 5020 1896 50  0000 L CNN
-F 1 "330R" H 5020 1805 50  0000 L CNN
+F 1 "470R" H 5020 1805 50  0000 L CNN
 F 2 "Resistor_SMD:R_1206_3216Metric_Pad1.42x1.75mm_HandSolder" V 4880 1850 50  0001 C CNN
 F 3 "~" H 4950 1850 50  0001 C CNN
@@
 P 5300 1850
 F 0 "R3" H 5370 1896 50  0000 L CNN
-F 1 "330R" H 5370 1805 50  0000 L CNN
+F 1 "220R" H 5370 1805 50  0000 L CNN
 F 2 "Resistor_SMD:R_1206_3216Metric_Pad1.42x1.75mm_HandSolder" V 5230 1850 50  0001 C CNN
 F 3 "~" H 5300 1850 50  0001 C CNN
@@
 P 5650 1850
 F 0 "R4" H 5720 1896 50  0000 L CNN
-F 1 "330R" H 5720 1805 50  0000 L CNN
+F 1 "100R" H 5720 1805 50  0000 L CNN
 F 2 "Resistor_SMD:R_1206_3216Metric_Pad1.42x1.75mm_HandSolder" V 5580 1850 50  0001 C CNN
 F 3 "~" H 5650 1850 50  0001 C CNN
@@
 P 6150 7200
 F 0 "C23" H 6268 7246 50  0000 L CNN
-F 1 "470µF" H 6268 7155 50  0000 L CNN
+F 1 "100µF" H 6268 7155 50  0000 L CNN
 F 2 "Capacitor_THT:CP_Radial_D6.3mm_P2.50mm" H 6188 7050 50  0001 C CNN
 F 3 "~" H 6150 7200 50  0001 C CNN
@@
 Wire Wire Line
 	9800 5100 9800 5150
+Text Notes 600  7000 0    50   ~ 0
+TODO: Rajouter des resistances de pulldown sur les entrées IN des BTN8982TA
 $EndSCHEMATC
