File: pcb/Carte_Chassis_DFRobotic/Carte_Chassis_DFRobotic.sch (KiCad schematic (older format))
At the start: 36 parts, among them J13 Conn_01x02, J5 Conn_02x07_Odd_Even, J6 Molex KK 254, J7 Samtec FTS-105-01-L-DV, J8 Samtec FTS-105-01-L-DV, Q1 NTR3C21NZT1G, SW1 SMR8016C-1, SW2 Reset, SW3 USER1, SW4 USER2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

Commit message: ajout de la carte chassi DFRobotics + creation d'une nouvelle carte led + creation d'une carte capteur pour DFRobotic + correction de l'alimentation en 5V des encodeurs sur DFRobotic (carte Landzo a corriger dans un prochaine commit)
Parts:
- removed C3: 100µF, Capacitor_THT:CP_Radial_D6.3mm_P2.50mm, symbol Device:CP
- removed C4: 100nF, Capacitor_SMD:C_1206_3216Metric_Pad1.42x1.75mm_HandSolder, symbol Device:C
- removed J5: Conn_02x07_Odd_Even, Connector_PinHeader_2.54mm:PinHeader_2x07_P2.54mm_Vertical, symbol Connector_Generic:Conn_02x07_Odd_Even
- removed J6: Molex KK 254, Connector_Molex:Molex_KK-254_AE-6410-04A_1x04_P2.54mm_Vertical, symbol Connector_Generic:Conn_01x04
- removed R10: 4.7K, Resistor_SMD:R_1206_3216Metric_Pad1.42x1.75mm_HandSolder, symbol Device:R
- removed R11: 2.2K, Resistor_SMD:R_1206_3216Metric_Pad1.42x1.75mm_HandSolder, symbol Device:R
- added C10, C11, C14, C15, C8, C9: 100nF, Capacitor_SMD:C_1206_3216Metric_Pad1.42x1.75mm_HandSolder, symbol Device:C
- added C13, C16: 1µF, Capacitor_SMD:C_1206_3216Metric_Pad1.42x1.75mm_HandSolder, symbol Device:C
- added J1, J14, J15, J17: Conn_01x03, Connector_PinHeader_2.54mm:PinHeader_1x03_P2.54mm_Horizontal, symbol Connector_Generic:Conn_01x03
- added J10, J9: DF3A-5P-2DS, Insa:DF3A-5P-2DS, symbol Connector_Generic:Conn_01x05
- added J11, J12: DF3A-4P-2DS, Insa:DF3A-4P-2DS, symbol Connector_Generic:Conn_01x04
- added J16: Conn_02x05_Odd_Even, Connector_Multicomp:Multicomp_MC9A12-1034_2x05_P2.54mm_Vertical, symbol Connector_Generic:Conn_02x05_Odd_Even
- added RN4, RN6: 2.2K, Resistor_SMD:R_Array_Convex_4x0603, symbol Device:R_Pack04
- added RN5, RN7: 3.3K, Resistor_SMD:R_Array_Convex_4x0603, symbol Device:R_Pack04
- added U5: MIC29500-3.3WT, Package_TO_SOT_THT:TO-220-3_Vertical, symbol Insa:MIC29500-3.3WT
- D1: footprint LED_THT:LED_D3.0mm -> LED_SMD:LED_1206_3216Metric_Pad1.42x1.75mm_HandSolder
Connections:
- net labels added: +5V, MOTOR_LEFT_PWM, MOTOR_RIGHT_PWM, SERVO_PWM2
- net labels removed: +BATT, DISABLE_MOT_L, DISABLE_MOT_R, FEEDBACK_MOT_L, FEEDBACK_MOT_R, PWM_MOT_L_1, PWM_MOT_L_2, PWM_MOT_R_1, PWM_MOT_R_2, VBAT_ADC
- wire segments 262 -> 329
- no-connect marks 32 -> 51
Other:
- note added: "ENC_SIG_A1 ->FTM_CLK0\nENC_SIG_A2 ->FTM_CLK1"
- note added: "Encoders"
- note added: "Pixy2"
- note added: "SERVO_PWM ->FTM0_CH4\nSERVO_PWM2 ->FTM0_CH5\nMOTOR_LEFT_PWM ->FTM0_CH1\nMOTOR_RIGHT_PWM ->FTM0_CH2\nPIXY2_UART -> UART1 (PTC3 et PTC4)"
- note added: "ToF Sensors"
- note added: "UART->UART0 (PTE20 et PTE21)\nSENS2 I2C ->I2C0\nSENS1 I2C ->I2C1"
- note removed: "FEEDBACK_L ->ADC_SE6\nFEEDBACK_R ->ADC_SE7\nENC_SIG_A1 ->FTM2_CH0\nENC_SIG_A2 ->FTM2_CH1"
- note removed: "SERVO_PWM ->FTM1_CH0\nPWM_MOT_Rx ->FTM0_CH1 et CH2\nPWM_MOT_Lx ->FTM0_CH4 et CH5"
- note removed: "VBAT_ADC->ADC0_SE3\nUART->UART0 (PTE20 et PTE21)\nSENS2 I2C ->I2C0\nSENS1 I2C ->I2C1"
- moved on the sheet: C1, C2, D1, R1
