File: pcb/DFRobotic/Carte_Chassis_DFRobotic/Carte_Chassis_DFRobotic.sch (KiCad schematic (older format))
At the start: 52 parts, among them J1 Conn_01x03, J10 DF3A-5P-2DS, J11 DF3A-4P-2DS, J12 DF3A-4P-2DS, J13 Conn_01x02, J14 Conn_01x03, J15 Conn_01x03, J16 Conn_02x05_Odd_Even, J17 Conn_01x03, J7 Samtec FTS-105-01-L-DV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

Commit message: Ajout des regles NXP Cup pour 2020 (V1) + modifs mineures sur pcbs
Parts:
- R1: value 100R -> 2.2K
Connections:
- net SW_USER2: now also U1.2.6 (PTD0); no longer U1.2.12 (PTD1)
Changed lines of the file:
@@
 Sheet 1 1
 Title "Carte_DFRobotic"
-Date "2020-01-29"
-Rev "1.0"
+Date "2020-02-03"
+Rev "1.1"
 Comp "INSA Toulouse (GEI)"
 Comment1 ""
@@
 P 2500 1200
 F 0 "R1" H 2570 1246 50  0000 L CNN
-F 1 "100R" H 2570 1155 50  0000 L CNN
+F 1 "2.2K" H 2570 1155 50  0000 L CNN
 F 2 "Resistor_SMD:R_1206_3216Metric_Pad1.42x1.75mm_HandSolder" V 2430 1200 50  0001 C CNN
 F 3 "~" H 2500 1200 50  0001 C CNN
@@
 	1500 6900 800  6900
 Wire Wire Line
-	4800 5400 5450 5400
+	4800 5100 5450 5100
 Wire Wire Line
 	4800 5300 5450 5300
 Text Label 5450 5300 2    50   ~ 0
 SW_USER1
-Text Label 5450 5400 2    50   ~ 0
+Text Label 5450 5100 2    50   ~ 0
 SW_USER2
 Wire Wire Line
@@
 NoConn ~ 2600 6300
 NoConn ~ 1500 5600
-NoConn ~ 4800 5100
 NoConn ~ 4800 5200
 NoConn ~ 4800 5600
@@
 Wire Wire Line
 	6100 4800 7150 4800
+NoConn ~ 4800 5400
 $EndSCHEMATC
