File: pcb/Generic/Carte_LED/Carte_LED.kicad_pcb (KiCad board)
At the start: 2 copper layers, 100 x 38 mm, 26 parts, among them J1 Conn_01x02, U1 ZLDO1117G50TA

Commit message: Ajout des regles NXP Cup pour 2020 (V1) + modifs mineures sur pcbs
Parts:
- added G1: LOGO, Insa:insa-image, F.Cu at (125.2, 73.9)
- R1, R2, R3, R4, R5, R6: value 10R -> 0R
