File: pcb/Generic/Carte_LED/Carte_LED.sch (KiCad schematic (older format))
At the start: 26 parts, among them J1 Conn_01x02, U1 ZLDO1117G50TA

Commit message: Ajout des regles NXP Cup pour 2020 (V1) + modifs mineures sur pcbs
Parts:
- added G1: LOGO, Insa:insa-image, symbol insa-sym:LOGO
- R1, R2, R3, R4, R5, R6: value 10R -> 0R
Other:
- note added: "VLCS5B30: 2.5V@35mA"
Changed lines of the file:
@@
 Sheet 1 1
 Title "Carte_LED"
-Date "2019-10-24"
-Rev "1.0"
+Date "2020-02-05"
+Rev "1.1"
 Comp "INSA GEI"
 Comment1 ""
@@
 P 2000 4450
 F 0 "R1" H 2070 4496 50  0000 L CNN
-F 1 "10R" H 2070 4405 50  0000 L CNN
+F 1 "0R" H 2070 4405 50  0000 L CNN
 F 2 "Resistor_THT:R_Axial_DIN0309_L9.0mm_D3.2mm_P2.54mm_Vertical" V 1930 4450 50  0001 C CNN
 F 3 "~" H 2000 4450 50  0001 C CNN
@@
 $EndComp
 $Comp
-L power:GND #PWR?
+L power:GND #PWR0105
 U 1 1 5E2F8E21
 P 5000 2050
-F 0 "#PWR?" H 5000 1800 50  0001 C CNN
+F 0 "#PWR0105" H 5000 1800 50  0001 C CNN
 F 1 "GND" H 5005 1877 50  0000 C CNN
 F 2 "" H 5000 2050 50  0001 C CNN
@@
 	5000 2000 5000 2050
 $Comp
-L power:+5V #PWR?
+L power:+5V #PWR0106
 U 1 1 5E2FC762
 P 6300 1050
-F 0 "#PWR?" H 6300 900 50  0001 C CNN
+F 0 "#PWR0106" H 6300 900 50  0001 C CNN
 F 1 "+5V" H 6315 1223 50  0000 C CNN
 F 2 "" H 6300 1050 50  0001 C CNN
@@
 	4400 1200 4400 1650
 $Comp
-L power:+5V #PWR?
+L power:+5V #PWR0107
 U 1 1 5E306037
 P 3100 4150
-F 0 "#PWR?" H 3100 4000 50  0001 C CNN
+F 0 "#PWR0107" H 3100 4000 50  0001 C CNN
 F 1 "+5V" H 3115 4323 50  0000 C CNN
 F 2 "" H 3100 4150 50  0001 C CNN
@@
 P 2450 4450
 F 0 "R2" H 2520 4496 50  0000 L CNN
-F 1 "10R" H 2520 4405 50  0000 L CNN
+F 1 "0R" H 2520 4405 50  0000 L CNN
 F 2 "Resistor_THT:R_Axial_DIN0309_L9.0mm_D3.2mm_P2.54mm_Vertical" V 2380 4450 50  0001 C CNN
 F 3 "~" H 2450 4450 50  0001 C CNN
@@
 P 2900 4450
 F 0 "R3" H 2970 4496 50  0000 L CNN
-F 1 "10R" H 2970 4405 50  0000 L CNN
+F 1 "0R" H 2970 4405 50  0000 L CNN
 F 2 "Resistor_THT:R_Axial_DIN0309_L9.0mm_D3.2mm_P2.54mm_Vertical" V 2830 4450 50  0001 C CNN
 F 3 "~" H 2900 4450 50  0001 C CNN
@@
 P 3300 4450
 F 0 "R4" H 3370 4496 50  0000 L CNN
-F 1 "10R" H 3370 4405 50  0000 L CNN
+F 1 "0R" H 3370 4405 50  0000 L CNN
 F 2 "Resistor_THT:R_Axial_DIN0309_L9.0mm_D3.2mm_P2.54mm_Vertical" V 3230 4450 50  0001 C CNN
 F 3 "~" H 3300 4450 50  0001 C CNN
@@
 P 3750 4450
 F 0 "R5" H 3820 4496 50  0000 L CNN
-F 1 "10R" H 3820 4405 50  0000 L CNN
+F 1 "0R" H 3820 4405 50  0000 L CNN
 F 2 "Resistor_THT:R_Axial_DIN0309_L9.0mm_D3.2mm_P2.54mm_Vertical" V 3680 4450 50  0001 C CNN
 F 3 "~" H 3750 4450 50  0001 C CNN
@@
 P 4200 4450
 F 0 "R6" H 4270 4496 50  0000 L CNN
-F 1 "10R" H 4270 4405 50  0000 L CNN
+F 1 "0R" H 4270 4405 50  0000 L CNN
 F 2 "Resistor_THT:R_Axial_DIN0309_L9.0mm_D3.2mm_P2.54mm_Vertical" V 4130 4450 50  0001 C CNN
 F 3 "~" H 4200 4450 50  0001 C CNN
@@
 Wire Wire Line
 	4200 4750 4200 4600
+Text Notes 900  4900 0    50   ~ 0
+VLCS5B30: 2.5V@35mA
+$Comp
+L insa-sym:LOGO G1
+U 1 1 5E3B0BBE
+P 7600 6800
+F 0 "G1" H 7600 6348 60  0001 C CNN
+F 1 "LOGO" H 7600 7252 60  0001 C CNN
+F 2 "Insa:insa-image" H 7600 6800 50  0001 C CNN
+F 3 "" H 7600 6800 50  0001 C CNN
+	1    7600 6800
+	1    0    0    -1
+$EndComp
 $EndSCHEMATC
