File: pcb/DFRobotic/Encodeurs-DFRobotics/Encodeurs-DFRobotics.sch (KiCad schematic (older format))
At the start: 12 parts, among them J1 DF3A-5P-2DS, J2 DF3A-5P-2DS, U1 AEDR-8300, U2 AEDR-8300, U3 74LVC2G34, U4 74LVC2G34

Commit message: Ajout des regles NXP Cup pour 2020 (V1) + modifs mineures sur pcbs
Parts:
- added G1: LOGO, symbol insa-sym:LOGO
Changed lines of the file:
@@
 Sheet 1 1
 Title "Encodeurs DFRobotics"
-Date "2020-01-30"
+Date "2020-02-05"
 Rev "1.0"
-Comp "INSA"
+Comp "INSA - GEI"
 Comment1 ""
 Comment2 ""
@@
 	2350 6950 2550 6950
 Connection ~ 2550 6950
+$Comp
+L insa-sym:LOGO G1
+U 1 1 5E3AFE48
+P 7600 6800
+F 0 "G1" H 7600 6348 60  0001 C CNN
+F 1 "LOGO" H 7600 7252 60  0001 C CNN
+F 2 "" H 7600 6800 50  0001 C CNN
+F 3 "" H 7600 6800 50  0001 C CNN
+	1    7600 6800
+	1    0    0    -1
+$EndComp
 $EndSCHEMATC

Commit message: Changement de capteur pour les encodeurs DFRobot
Parts:
- removed C1, C2: 1µF, Capacitor_SMD:C_0805_2012Metric_Pad1.15x1.40mm_HandSolder, symbol Device:C
- removed U1, U2: AEDR-8300, Insa:AEDR-8300, symbol Insa:AEDR-3800
- added R3, R4: 200, Resistor_SMD:R_0805_2012Metric_Pad1.15x1.40mm_HandSolder, symbol Device:R
- added U1, U2: SFH9206, OptoDevice:Osram_SFH9x0x, symbol Sensor_Proximity:SFH9206
Connections:
- net +5V: now also R1.2, R2.2, R3.1, R4.1; no longer R1.1, R2.1
- net GND: now also J1.4 (Pin_4), J2.4 (Pin_4), U3.3, U4.3, U1.3 (E), U1.6 (K), U2.3 (E), U2.6 (K)
- net at U3.1: now also R3.2, U1.4 (C)
- net at U4.1: now also R4.2, U2.4 (C)
- net SENS_LEFT_B: no longer names the net of U3.4
- net SENS_LEFT_B: no longer J1.4 (Pin_4)
- net SENS_RIGHT_B: no longer names the net of U4.4
- net SENS_RIGHT_B: no longer J2.4 (Pin_4)
- new net: R1.1, U1.1 (A)
- new net: R2.1, U2.1 (A)
- no-connect marks 0 -> 2
Other:
- moved on the sheet: R1, R2
